File: Magnetometer_Board_Kicad/Magnetometer_Board_Kicad.kicad_sch (KiCad schematic)
At the start: 18 parts, among them J1 JST_SH_10pin, J2 +5V pad, J3 GND pad, U1 IST8310, U2 TPS77033PDBV, U3 TPS77033PDBV

Commit message: production files done
Parts:
- C1, C2, C6, C7: LCSC (none) -> C77046
- C3, C5: LCSC (none) -> C77055
- C4: value 100n -> 4.7u; LCSC (none) -> C327022
- D1, D2: LCSC (none) -> C1869319
- J1: LCSC (none) -> C160409
- R1, R2, R3: LCSC (none) -> C95177
- U1: LCSC (none) -> C2683055; LCSC number C2683055 -> (none)
- U2, U3: LCSC (none) -> C36996065
